Commit message: feat: lidar module completed

File: description/lidar.xacro (robot description, xacro)
@@ -4,5 +4,5 @@
         <parent link="chassis"/>
         <child link="laser_frame"/>
-        <origin xyz="0.64 0 0.315" rpy="0 0 0"/>
+        <origin xyz="0.560407 0 0.385" rpy="0 0 0"/>
     </joint>
     <link name="laser_frame">
@@ -10,4 +10,11 @@
             <geometry>
                 <cylinder radius="0.05" length="0.04"/>
+            </geometry>
+            <material name="red"/>
+        </visual>
+        <visual>
+            <origin xyz="0 0 -0.05"/>
+            <geometry>
+                <cylinder radius="0.01" length="0.1"/>
             </geometry>
             <material name="red"/>
@@ -24,28 +31,31 @@
     <gazebo reference="laser_frame">
         <material>Gazebo/Red</material>
-        <sensor name="laser" type="ray">
-            <pose> 0 0 0 0 0 0 </pose>
-            <visualize>false</visualize>
-            <update_rate>10</update_rate>
+        <sensor name='laser_frame' type='gpu_lidar'>
+            <pose relative_to='laser_frame'>0 0 0 0 0 0</pose>
+            <topic>scan</topic>
+            <update_rate>20</update_rate>
             <ray>
                 <scan>
                     <horizontal>
-                        <samples>360</samples>
-                        <min_angle>-3.14</min_angle>
-                        <max_angle>3.14</max_angle>
+                        <samples>120</samples>
+                        <resolution>1</resolution>
+                        <min_angle>-3.14159</min_angle> <!-- -π radians -->
+                        <max_angle>3.14159</max_angle>
                     </horizontal>
+                    <vertical>
+                        <samples>10</samples>
+                        <resolution>1</resolution>
+                        <min_angle>-0.262</min_angle>
+                        <max_angle>0.262</max_angle>
+                    </vertical>
                 </scan>
                 <range>
-                    <min>0.3</min>
-                    <max>12</max>
+                    <min>0.1</min>
+                    <max>5.0</max>
+                    <resolution>0.1</resolution>
                 </range>
             </ray>
-            <plugin name="laser_controller" filename="libgazebo_ros_ray_sensor.so">
-                <ros>
-                    <argument>~/out:=scan</argument>
-                </ros>
-                <output_type>sensor_msgs/LaserScan</output_type>
-                <frame_name>laser_frame</frame_name>
-            </plugin>
+            <always_on>1</always_on>
+            <visualize>true</visualize>
         </sensor>
     </gazebo>

File: description/robot.urdf.xacro (robot description, xacro)
@@ -10,5 +10,5 @@
         <xacro:include filename="gazebo_control.xacro" />
     </xacro:unless>
-    <!--<xacro:include filename="lidar.xacro" />-->
+    <xacro:include filename="lidar.xacro" />
     <!--<xacro:include filename="depth_camera.xacro" />-->
     <!-- <xacro:include filename="camera.xacro" /> -->

File: description/robot_visual.xacro (robot description, xacro)
@@ -92,5 +92,5 @@
         <material name="blue"/>
       </visual>
-      <!-- velodyne_vlp16 -->
+      <!-- velodyne_vlp16
       <visual>
         <origin xyz="0.560407 0.0981063 -0.282354" rpy="-4.83258e-15 6.44901e-15 -0.612605"/>
@@ -100,4 +100,5 @@
         <material name="red"/>
       </visual>
+      -->
       <!-- bort_motor (upper assembly) -->
       <visual>
