Commit message: Trying to create virtual infinite lines

File: src/esda_simulation_2025/description/camera.xacro (robot description, xacro)
@@ -28,4 +28,11 @@
         -->
     </link>
+    <!-- IMU built into the ZED camera -->
+    <joint name="imu_joint" type="fixed">
+        <parent link="camera_link"/>
+        <child link="imu_link"/>
+        <origin xyz="0 0 0" rpy="0 0 0"/>
+    </joint>
+    <link name="imu_link"/>
     <joint name="camera_optical_joint" type="fixed">
         <parent link="camera_link"/>
@@ -106,3 +113,10 @@
         </sensor>
     </gazebo>
+    <gazebo reference="imu_link">
+        <sensor name="zed_imu" type="imu">
+            <always_on>true</always_on>
+            <update_rate>100</update_rate>
+            <topic>imu/data</topic>
+        </sensor>
+    </gazebo>
 </robot>

Commit message: Reverted back to commit hash [200~470b7eb

File: src/esda_simulation_2025/description/camera.xacro (robot description, xacro)
@@ -28,11 +28,4 @@
         -->
     </link>
-    <!-- IMU built into the ZED camera -->
-    <joint name="imu_joint" type="fixed">
-        <parent link="camera_link"/>
-        <child link="imu_link"/>
-        <origin xyz="0 0 0" rpy="0 0 0"/>
-    </joint>
-    <link name="imu_link"/>
     <joint name="camera_optical_joint" type="fixed">
         <parent link="camera_link"/>
@@ -113,10 +106,3 @@
         </sensor>
     </gazebo>
-    <gazebo reference="imu_link">
-        <sensor name="zed_imu" type="imu">
-            <always_on>true</always_on>
-            <update_rate>100</update_rate>
-            <topic>imu/data</topic>
-        </sensor>
-    </gazebo>
 </robot>

Commit message: Testing with the increased ZedCam height

File: src/esda_simulation_2025/description/camera.xacro (robot description, xacro)
@@ -1,9 +1,41 @@
 <?xml version="1.0"?>
 <robot xmlns:xacro="http://www.ros.org/wiki/xacro" >
-    <joint name="camera_joint" type="fixed">
-        <parent link="chassis"/>
-        <child link="camera_link"/>
-        <origin xyz="0.8 0 0.315" rpy="0 0 0"/> <!--TODO: need to change to our actual camera location. the 0.005 is because the camera has a thickness-->
-    </joint>
+    <!-- camera_mount: "front" (default) is the original low, forward-facing
+         mount. "pole_top" mounts the camera on the LiDAR pole (lidar.xacro),
+         just below the LiDAR itself. Select with e.g.
+         `xacro robot.urdf.xacro camera_mount:=pole_top`.
+         x below MUST match lidar_mount_x in lidar.xacro - that's the pole's
+         actual x station on our chassis. (The raw xyz from
+         assets/robot_pruned.urdf's ZED placement can't be reused directly:
+         that file's "chassis" origin is a different reference point than
+         ours - copying its numbers put the camera at the back of the robot
+         instead of on the pole.)
+         y is offset off the pole's own y=0 (a short side bracket) rather
+         than sharing it exactly - otherwise the camera sits directly behind
+         the LiDAR in every view instead of beside it.
+         The CAD reference's rpy put its 15 deg tilt on roll (rpy="0.266 0 0"),
+         which only spins the image about the boresight - it doesn't tilt the
+         camera up/down. A downward tilt is pitch (rotation about Y): with
+         ROS's X-forward/Z-up convention, positive pitch tips +X toward -Z,
+         i.e. downward. -->
+    <xacro:arg name="camera_mount" default="front" />
+    <xacro:if value="${'$(arg camera_mount)' == 'pole_top'}">
+        <joint name="camera_joint" type="fixed">
+            <parent link="chassis"/>
+            <child link="camera_link"/>
+            <!-- x = lidar_mount_x (0.560407); y = +0.10 (side bracket off the
+                 pole); z = 1.30, ~8.5cm below the pole-top LiDAR
+                 (lidar_pole_base_z 0.385 + lidar_pole_length 1.0 = 1.385);
+                 pitch = 15 deg down (see note above) -->
+            <origin xyz="0.560407 0.10 1.30" rpy="0 0.2618 0"/>
+        </joint>
+    </xacro:if>
+    <xacro:unless value="${'$(arg camera_mount)' == 'pole_top'}">
+        <joint name="camera_joint" type="fixed">
+            <parent link="chassis"/>
+            <child link="camera_link"/>
+            <origin xyz="0.8 0 0.315" rpy="0 0 0"/> <!--TODO: need to change to our actual camera location. the 0.005 is because the camera has a thickness-->
+        </joint>
+    </xacro:unless>
     <link name="camera_link">
         <visual>

File: src/esda_simulation_2025/description/lidar.xacro (robot description, xacro)
@@ -1,9 +1,63 @@
 <?xml version="1.0"?>
 <robot xmlns:xacro="http://www.ros.org/wiki/xacro" >
-    <joint name="laser_joint" type="fixed">
-        <parent link="chassis"/>
-        <child link="laser_frame"/>
-        <origin xyz="0.560407 0 0.385" rpy="0 0 0"/>
-    </joint>
+    <!-- lidar_mount: "pole_top" (default) raises the sensor on a mounting
+         pole above the chassis/camera so its 360 deg scan isn't blocked.
+         "low" reverts to the original single mount, directly on the chassis,
+         no pole. Select with e.g. `xacro robot.urdf.xacro lidar_mount:=low`.
+         camera.xacro's "pole_top" camera_mount option assumes this pole
+         exists (it reuses lidar_mount_x as its own x) - pairing
+         camera_mount:=pole_top with lidar_mount:=low doesn't make physical
+         sense (there is no pole to mount it on). -->
+    <xacro:arg name="lidar_mount" default="pole_top" />
+    <!-- Pole: square tube, sized to match the physical part
+         (assets/pruned/part_1__7.stl is 40x40mm x 1.0m). The base sits at
+         the old (pre-pole) sensor mount point; the sensor itself sits on
+         top of the pole, 1m higher, at the same x/y. -->
+    <xacro:property name="lidar_pole_width"  value="0.04"/>
+    <xacro:property name="lidar_pole_length" value="1.0"/>
+    <xacro:property name="lidar_pole_mass"   value="0.3"/>
+    <xacro:property name="lidar_mount_x"     value="0.560407"/>
+    <xacro:property name="lidar_mount_y"     value="0"/>
+    <xacro:property name="lidar_pole_base_z" value="0.385"/>
+    <xacro:if value="${'$(arg lidar_mount)' == 'pole_top'}">
+        <joint name="lidar_pole_joint" type="fixed">
+            <parent link="chassis"/>
+            <child link="lidar_pole"/>
+            <origin xyz="${lidar_mount_x} ${lidar_mount_y} ${lidar_pole_base_z}" rpy="0 0 0"/>
+        </joint>
+        <link name="lidar_pole">
+            <visual>
+                <origin xyz="0 0 ${lidar_pole_length/2}"/>
+                <geometry>
+                    <box size="${lidar_pole_width} ${lidar_pole_width} ${lidar_pole_length}"/>
+                </geometry>
+                <material name="grey"/>
+            </visual>
+            <collision>
+                <origin xyz="0 0 ${lidar_pole_length/2}"/>
+                <geometry>
+                    <box size="${lidar_pole_width} ${lidar_pole_width} ${lidar_pole_length}"/>
+                </geometry>
+            </collision>
+            <xacro:inertial_box mass="${lidar_pole_mass}" x="${lidar_pole_width}" y="${lidar_pole_width}" z="${lidar_pole_length}">
+                <origin xyz="0 0 ${lidar_pole_length/2}" rpy="0 0 0"/>
+            </xacro:inertial_box>
+        </link>
+        <gazebo reference="lidar_pole">
+            <material>Gazebo/Grey</material>
+        </gazebo>
+        <joint name="laser_joint" type="fixed">
+            <parent link="lidar_pole"/>
+            <child link="laser_frame"/>
+            <origin xyz="0 0 ${lidar_pole_length}" rpy="0 0 0"/>
+        </joint>
+    </xacro:if>
+    <xacro:unless value="${'$(arg lidar_mount)' == 'pole_top'}">
+        <joint name="laser_joint" type="fixed">
+            <parent link="chassis"/>
+            <child link="laser_frame"/>
+            <origin xyz="${lidar_mount_x} ${lidar_mount_y} ${lidar_pole_base_z}" rpy="0 0 0"/>
+        </joint>
+    </xacro:unless>
     <link name="laser_frame">
         <visual>

File: src/esda_simulation_2025/description/ros2_control_2wd.xacro (robot description, xacro)
@@ -3,4 +3,8 @@
   <xacro:arg name="namespace" default="" />
   <xacro:arg name="sim_mode" default="false" />
+  <!-- Overridable so launch_hardware.launch.py can point this at the ESP32
+       (typically /dev/ttyUSB0) instead of the STM32's /dev/ttyACM0. -->
+  <xacro:arg name="serial_device" default="/dev/ttyACM0" />
+  <xacro:arg name="serial_baud_rate" default="57600" />
   <!--
   <xacro:unless value="$(arg sim_mode)">
@@ -27,6 +31,6 @@
         <param name="right_wheel_name">right_wheel_joint</param>
         <param name="loop_rate">30</param>
-        <param name="device">/dev/ttyACM0</param>
-        <param name="baud_rate">57600</param>
+        <param name="device">$(arg serial_device)</param>
+        <param name="baud_rate">$(arg serial_baud_rate)</param>
         <param name="timeout_ms">1000</param>
         <param name="open_loop">false</param>

Commit message: Added a new configuration where the zed cam is placed at the current position on the real robot (in front of the lidar on the chassis)

File: src/esda_simulation_2025/description/camera.xacro (robot description, xacro)
@@ -3,6 +3,9 @@
     <!-- camera_mount: "front" (default) is the original low, forward-facing
          mount. "pole_top" mounts the camera on the LiDAR pole (lidar.xacro),
-         just below the LiDAR itself. Select with e.g.
-         `xacro robot.urdf.xacro camera_mount:=pole_top`.
+         just below the LiDAR itself. "top_front" is the real robot as
+         photographed: the ZED on a short bracket above the red beacon, on
+         the top deck just in front of the Velodyne (pair it with
+         lidar_mount:=low, which is how that robot carries its LiDAR).
+         Select with e.g. `xacro robot.urdf.xacro camera_mount:=top_front`.
          x below MUST match lidar_mount_x in lidar.xacro - that's the pole's
          actual x station on our chassis. (The raw xyz from
@@ -31,5 +34,18 @@
         </joint>
     </xacro:if>
-    <xacro:unless value="${'$(arg camera_mount)' == 'pole_top'}">
+    <xacro:if value="${'$(arg camera_mount)' == 'top_front'}">
+        <joint name="camera_joint" type="fixed">
+            <parent link="chassis"/>
+            <child link="camera_link"/>
+            <!-- Estimated from photos of the real robot, NOT measured:
+                 x = 0.76, ~20 cm in front of the low LiDAR (lidar_mount_x
+                 0.560407); y = 0, on the centreline; z = 0.41, ~11 cm above
+                 the top deck (chassis_height 0.30) on the bracket over the
+                 beacon; level (no visible tilt). Replace with tape-measure
+                 values from the chassis origin when available. -->
+            <origin xyz="0.76 0 0.41" rpy="0 0 0"/>
+        </joint>
+    </xacro:if>
+    <xacro:unless value="${'$(arg camera_mount)' in ('pole_top', 'top_front')}">
         <joint name="camera_joint" type="fixed">
             <parent link="chassis"/>
